File: MyProjects/Office Clock/Office Clock.sch (EAGLE design)
At the start: 1 part, among them IC1 74HC164N

Commit message: Office Clock WIP
Parts:
- added IC2, IC3, IC5, IC6: MAX7219CNG, maxim:MAX7219CNG
- added IC4: 74HCT164D, 74xx-us:74HCT164D
- added JP1: (no value), pinhead:PINHD-1X2
- added T1: SFH303, opto-trans-siemens:SFH303
- added U$1, U$2, U$3, U$4: YSM-1288CR3G2C, led-matrix-v3:YSM-1288CR3G2C
- added U$5, U$6: DLX3416, DLX3416:DLX3416
- added WEMOS1: (no value), esp8266modules:WEMOS-D1-MINI
- IC1: value 74HC164N -> 74LS126D; device 74xx-us:74HC164N -> 74xx-us:74LS126D
Changed lines of the file:
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@@
 </classes>
 <parts>
-<part name="IC1" library="74xx-us" library_urn="urn:adsk.eagle:library:88" deviceset="74*164" device="N" package3d_urn="urn:adsk.eagle:package:2921/1" technology="HC"/>
+<part name="WEMOS1" library="esp8266modules" deviceset="WEMOS-D1-MINI" device=""/>
+<part name="IC2" library="maxim" library_urn="urn:adsk.eagle:library:269" deviceset="MAX7219CNG" device="" package3d_urn="urn:adsk.eagle:package:17515/1"/>
+<part name="IC4" library="74xx-us" library_urn="urn:adsk.eagle:library:88" deviceset="74*164" device="D" package3d_urn="urn:adsk.eagle:package:2917/1" technology="HCT"/>
+<part name="IC1" library="74xx-us" library_urn="urn:adsk.eagle:library:88" deviceset="74*126" device="D" package3d_urn="urn:adsk.eagle:package:2917/1" technology="LS"/>
+<part name="U$1" library="led-matrix-v3" deviceset="YSM-1288CR3G2C" device=""/>
+<part name="U$2" library="led-matrix-v3" deviceset="YSM-1288CR3G2C" device=""/>
+<part name="U$3" library="led-matrix-v3" deviceset="YSM-1288CR3G2C" device=""/>
+<part name="U$4" library="led-matrix-v3" deviceset="YSM-1288CR3G2C" device=""/>
+<part name="IC3" library="maxim" library_urn="urn:adsk.eagle:library:269" deviceset="MAX7219CNG" device="" package3d_urn="urn:adsk.eagle:package:17515/1"/>
+<part name="IC5" library="maxim" library_urn="urn:adsk.eagle:library:269" deviceset="MAX7219CNG" device="" package3d_urn="urn:adsk.eagle:package:17515/1"/>
+<part name="IC6" library="maxim" library_urn="urn:adsk.eagle:library:269" deviceset="MAX7219CNG" device="" package3d_urn="urn:adsk.eagle:package:17515/1"/>
+<part name="U$5" library="DLX3416" deviceset="DLX3416" device=""/>
+<part name="U$6" library="DLX3416" deviceset="DLX3416" device=""/>
+<part name="T1" library="opto-trans-siemens" library_urn="urn:adsk.eagle:library:317" deviceset="SFH303" device="" package3d_urn="urn:adsk.eagle:package:21797/1"/>
+<part name="JP1" library="pinhead" library_urn="urn:adsk.eagle:library:325" deviceset="PINHD-1X2" device="" package3d_urn="urn:adsk.eagle:package:22435/2"/>
 </parts>
 <sheets>
@@
 </plain>
 <instances>
-<instance part="IC1" gate="A" x="50.8" y="63.5"/>
+<instance part="WEMOS1" gate="D1" x="-66.04" y="83.82"/>
+<instance part="IC2" gate="G$1" x="15.24" y="88.9"/>
+<instance part="IC4" gate="A" x="76.2" y="2.54"/>
+<instance part="IC1" gate="A" x="-27.94" y="99.06"/>
+<instance part="IC1" gate="B" x="-27.94" y="73.66"/>
+<instance part="IC1" gate="C" x="-27.94" y="50.8"/>
+<instance part="IC1" gate="D" x="-27.94" y="20.32"/>
+<instance part="U$1" gate="G$1" x="12.7" y="147.32"/>
+<instance part="U$2" gate="G$1" x="50.8" y="147.32"/>
+<instance part="U$3" gate="G$1" x="96.52" y="147.32"/>
+<instance part="U$4" gate="G$1" x="142.24" y="147.32"/>
+<instance part="IC3" gate="G$1" x="53.34" y="88.9"/>
+<instance part="IC5" gate="G$1" x="99.06" y="88.9"/>
+<instance part="IC6" gate="G$1" x="144.78" y="88.9"/>
+<instance part="U$5" gate="G$1" x="63.5" y="33.02"/>
+<instance part="U$6" gate="G$1" x="124.46" y="33.02"/>
+<instance part="T1" gate="G$1" x="-66.04" y="45.72"/>
+<instance part="JP1" gate="G$1" x="-63.5" y="20.32"/>
 </instances>
 <busses>
@@
 </drawing>
 <compatibility>
+<note version="6.3" minversion="6.2.2" severity="warning">
+Since Version 6.2.2 text objects can contain more than one line,
+which will not be processed correctly with this version.
+</note>
 <note version="8.2" severity="warning">
 Since Version 8.2, EAGLE supports online libraries. The ids

Commit message: Updates to Office Clock
Parts:
- removed IC4: 74HCT164D, 74xx-us:74HCT164D
- removed IC5, IC6: MAX7219CNG, maxim:MAX7219CNG
- added LED1, LED2: (no value), led:LED3MM
- IC1: value 74LS126D -> 74367N; device 74xx-us:74LS126D -> 74xx-us:74367N
- IC3: value MAX7219CNG -> 74HCT164N; device maxim:MAX7219CNG -> 74xx-us:74HCT164N
- U$1, U$2, U$4: value YSM-1288CR3G2C -> LN518GA; device led-matrix-v3:YSM-1288CR3G2C -> MyDisplays:LN518XX
- U$3: value YSM-1288CR3G2C -> LN518XGA; device led-matrix-v3:YSM-1288CR3G2C -> MyDisplays:LN518XX
Other:
- moved on the sheet: IC2
Changed lines of the file:
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@@
 <layer number="18" name="Vias" color="2" fill="1" visible="no" active="no"/>
 <layer number="19" name="Unrouted" color="6" fill="1" visible="no" active="no"/>
-<layer number="20" name="Dimension" color="15" fill="1" visible="no" active="no"/>
+<layer number="20" name="Dimension" color="24" fill="1" visible="no" active="no"/>
 <layer number="21" name="tPlace" color="7" fill="1" visible="no" active="no"/>
 <layer number="22" name="bPlace" color="7" fill="1" visible="no" active="no"/>
@@
 <layer number="48" name="Document" color="7" fill="1" visible="no" active="no"/>
 <layer number="49" name="Reference" color="7" fill="1" visible="no" active="no"/>
-<layer number="51" name="tDocu" color="6" fill="1" visible="no" active="no"/>
+<layer number="51" name="tDocu" color="7" fill="1" visible="no" active="no"/>
 <layer number="52" name="bDocu" color="7" fill="1" visible="no" active="no"/>
 <layer number="88" name="SimResults" color="9" fill="1" visible="yes" active="yes"/>
@@
 <part name="WEMOS1" library="esp8266modules" deviceset="WEMOS-D1-MINI" device=""/>
 <part name="IC2" library="maxim" library_urn="urn:adsk.eagle:library:269" deviceset="MAX7219CNG" device="" package3d_urn="urn:adsk.eagle:package:17515/1"/>
-<part name="IC4" library="74xx-us" library_urn="urn:adsk.eagle:library:88" deviceset="74*164" device="D" package3d_urn="urn:adsk.eagle:package:2917/1" technology="HCT"/>
-<part name="IC1" library="74xx-us" library_urn="urn:adsk.eagle:library:88" deviceset="74*126" device="D" package3d_urn="urn:adsk.eagle:package:2917/1" technology="LS"/>
-<part name="U$1" library="led-matrix-v3" deviceset="YSM-1288CR3G2C" device=""/>
-<part name="U$2" library="led-matrix-v3" deviceset="YSM-1288CR3G2C" device=""/>
-<part name="U$3" library="led-matrix-v3" deviceset="YSM-1288CR3G2C" device=""/>
-<part name="U$4" library="led-matrix-v3" deviceset="YSM-1288CR3G2C" device=""/>
-<part name="IC3" library="maxim" library_urn="urn:adsk.eagle:library:269" deviceset="MAX7219CNG" device="" package3d_urn="urn:adsk.eagle:package:17515/1"/>
-<part name="IC5" library="maxim" library_urn="urn:adsk.eagle:library:269" deviceset="MAX7219CNG" device="" package3d_urn="urn:adsk.eagle:package:17515/1"/>
-<part name="IC6" library="maxim" library_urn="urn:adsk.eagle:library:269" deviceset="MAX7219CNG" device="" package3d_urn="urn:adsk.eagle:package:17515/1"/>
 <part name="U$5" library="DLX3416" deviceset="DLX3416" device=""/>
 <part name="U$6" library="DLX3416" deviceset="DLX3416" device=""/>
 <part name="T1" library="opto-trans-siemens" library_urn="urn:adsk.eagle:library:317" deviceset="SFH303" device="" package3d_urn="urn:adsk.eagle:package:21797/1"/>
 <part name="JP1" library="pinhead" library_urn="urn:adsk.eagle:library:325" deviceset="PINHD-1X2" device="" package3d_urn="urn:adsk.eagle:package:22435/2"/>
+<part name="U$1" library="MyDisplays" deviceset="LN518XX" device="" value="LN518GA"/>
+<part name="U$2" library="MyDisplays" deviceset="LN518XX" device="" value="LN518GA"/>
+<part name="U$3" library="MyDisplays" deviceset="LN518XX" device="" value="LN518XGA"/>
+<part name="U$4" library="MyDisplays" deviceset="LN518XX" device="" value="LN518GA"/>
+<part name="IC1" library="74xx-us" library_urn="urn:adsk.eagle:library:88" deviceset="74*367" device="N" package3d_urn="urn:adsk.eagle:package:2922/1"/>
+<part name="IC3" library="74xx-us" library_urn="urn:adsk.eagle:library:88" deviceset="74*164" device="N" package3d_urn="urn:adsk.eagle:package:2921/1" technology="HCT"/>
+<part name="LED1" library="led" library_urn="urn:adsk.eagle:library:259" deviceset="LED" device="3MM" package3d_urn="urn:adsk.eagle:package:15797/1"/>
+<part name="LED2" library="led" library_urn="urn:adsk.eagle:library:259" deviceset="LED" device="3MM" package3d_urn="urn:adsk.eagle:package:15797/1"/>
 </parts>
 <sheets>
@@
 <instances>
 <instance part="WEMOS1" gate="D1" x="-66.04" y="83.82"/>
-<instance part="IC2" gate="G$1" x="15.24" y="88.9"/>
-<instance part="IC4" gate="A" x="76.2" y="2.54"/>
-<instance part="IC1" gate="A" x="-27.94" y="99.06"/>
-<instance part="IC1" gate="B" x="-27.94" y="73.66"/>
-<instance part="IC1" gate="C" x="-27.94" y="50.8"/>
-<instance part="IC1" gate="D" x="-27.94" y="20.32"/>
-<instance part="U$1" gate="G$1" x="12.7" y="147.32"/>
-<instance part="U$2" gate="G$1" x="50.8" y="147.32"/>
-<instance part="U$3" gate="G$1" x="96.52" y="147.32"/>
-<instance part="U$4" gate="G$1" x="142.24" y="147.32"/>
-<instance part="IC3" gate="G$1" x="53.34" y="88.9"/>
-<instance part="IC5" gate="G$1" x="99.06" y="88.9"/>
-<instance part="IC6" gate="G$1" x="144.78" y="88.9"/>
+<instance part="IC2" gate="G$1" x="25.4" y="81.28"/>
 <instance part="U$5" gate="G$1" x="63.5" y="33.02"/>
 <instance part="U$6" gate="G$1" x="124.46" y="33.02"/>
 <instance part="T1" gate="G$1" x="-66.04" y="45.72"/>
 <instance part="JP1" gate="G$1" x="-63.5" y="20.32"/>
+<instance part="U$1" gate="G$1" x="-55.88" y="149.86"/>
+<instance part="U$2" gate="G$1" x="-25.4" y="149.86"/>
+<instance part="U$3" gate="G$1" x="5.08" y="149.86"/>
+<instance part="U$4" gate="G$1" x="35.56" y="149.86"/>
+<instance part="IC1" gate="A" x="-25.4" y="81.28"/>
+<instance part="IC3" gate="A" x="-5.08" y="38.1"/>
+<instance part="LED1" gate="G$1" x="-10.16" y="152.4"/>
+<instance part="LED2" gate="G$1" x="-10.16" y="137.16"/>
 </instances>
 <busses>
+<bus name="SEGMENT[0..7]">
+<segment>
+<wire x1="-73.66" y1="154.94" x2="-73.66" y2="127" width="0.762" layer="92"/>
+<wire x1="-73.66" y1="127" x2="20.32" y2="127" width="0.762" layer="92"/>
+</segment>
+</bus>
 </busses>
 <nets>
